Commit message: CheackPoint2

File: my_rb1_description/urdf/my_rb1_robot.urdf (robot description, URDF)
Before this commit: robot my_rb1_robot, 7 links, 6 joints
Links:
- link back_caster: geometry collision sphere radius=0.010; collision sphere radius=0.025
- link base_footprint: mass None -> 0.0
- link front_caster: geometry collision sphere radius=0.010; collision sphere radius=0.025
- link front_laser: mass None -> 0.5; geometry collision cylinder length=0.10 radius=0.05; visual cylinder length=0.10 radius=0.05
- link left_wheel: geometry collision cylinder length=0.03 radius=0.025; visual cylinder length=0.03 radius=0.025
- link right_wheel: geometry collision cylinder length=0.03 radius=0.025; visual cylinder length=0.03 radius=0.025
Joints:
- removed joint back_caster_joint
- removed joint base_footprint_joint
- removed joint front_caster_joint
- removed joint front_laser_joint
- removed joint left_wheel_joint
- removed joint right_wheel_joint
- added joint joint_back_chassis_caster_wheel: type fixed, parent base_link, child back_caster, origin xyz=-0.1 0.0 -0.15 rpy=0 0 0
- added joint joint_base_link: type fixed, parent base_footprint, child base_link, origin xyz=0.0 0.0 0.15 rpy=0 0 0
- added joint joint_chassis_left_wheel: type continuous, parent base_link, child left_wheel, origin xyz=0.0 0.2 -0.15 rpy=0 0 0, axis 0 1 0, limit effort=10000 velocity=1000
- added joint joint_chassis_right_wheel: type continuous, parent base_link, child right_wheel, origin xyz=0.0 -0.2 -0.15 rpy=0 0 0, axis 0 1 0, limit effort=10000 velocity=1000
- added joint joint_front_chassis_caster_wheel: type fixed, parent base_link, child front_caster, origin xyz=0.1 0.0 -0.15 rpy=0 0 0
- added joint joint_laser_scan_chassis: type fixed, parent base_link, child front_laser, origin xyz=0.25 0.0 0.075 rpy=3.14 0 0
